Commit message: updated the flexiv model

File: urdf_models/flexiv_violin/flexiv.urdf (robot description, URDF)
Before this commit: robot 4S-Titania, 10 links, 9 joints
Links:
- link link1: geometry visual mesh filename=meshes/rizon4s/visual/link1.obj; visual mesh filename=meshes/rizon4s/visual/ring.obj scale=0.062 0.062 0.002
- link link2: geometry visual mesh filename=meshes/rizon4s/visual/link2.obj; visual mesh filename=meshes/rizon4s/visual/ring.obj scale=0.062 0.062 0.002
- link link3: geometry visual mesh filename=meshes/rizon4s/visual/link3.obj; visual mesh filename=meshes/rizon4s/visual/ring.obj scale=0.051 0.051 0.002
- link link4: geometry visual mesh filename=meshes/rizon4s/visual/link4.obj; visual mesh filename=meshes/rizon4s/visual/ring.obj scale=0.051 0.051 0.002
- link link5: geometry visual mesh filename=meshes/rizon4s/visual/link5.obj; visual mesh filename=meshes/rizon4s/visual/ring.obj scale=0.051 0.051 0.002
- link link6: geometry visual mesh filename=meshes/rizon4s/visual/link6.obj; visual mesh filename=meshes/rizon4s/visual/ring.obj scale=0.051 0.051 0.002
- link link7: geometry visual mesh filename=meshes/rizon4s/visual/link7.obj; visual mesh filename=meshes/rizon4s/visual/ring.obj scale=0.051 0.051 0.002
Joints:
- joint bow_joint: origin xyz=0.35 0 0.2 rpy=-1.57 0 1.57 -> xyz=-0.35 0 0.1 rpy=-1.57 0 -1.57; parent link7 -> flange
- joint joint7: origin xyz=-0.055 0.07 0.11 rpy=0.0 -1.5707963478683205 0.0 -> xyz=-0.015 0.07 0.11 rpy=0.0 -1.5707963478683205 0.0

Commit message: first try adding sound in the sim

File: urdf_models/flexiv_violin/flexiv.urdf (robot description, URDF)
Before this commit: robot 4S-Titania, 10 links, 9 joints
Links:
- link bow: mass 1.0 -> 0.06
- link link7: geometry collision mesh filename=meshes/rizon4s/collision/link7.stl; visual mesh filename=meshes/rizon4s/visual/link7.obj
