Commit message: coded two state machines, bowing + calibration, without any transition between the strings. Commented the sound + control sphere to avoid needing to change core functions in opensai.

File: urdf_models/flexiv_violin/violin.urdf (robot description, URDF)
Before this commit: robot violin, 5 links, 4 joints
Links:
- removed link cord1
- removed link cord2
- removed link cord3
- removed link cord4
- added link string1, mass 0.1; collision cylinder length=0.33 radius=0.001; visual cylinder length=0.33 radius=0.001
- added link string2, mass 0.1; collision cylinder length=0.33 radius=0.001; visual cylinder length=0.33 radius=0.001
- added link string3, mass 0.1; collision cylinder length=0.33 radius=0.001; visual cylinder length=0.33 radius=0.001
- added link string4, mass 0.1; collision cylinder length=0.33 radius=0.001; visual cylinder length=0.33 radius=0.001
- link base_link: geometry collision box size=0.2 0.5 0.01; visual box size=0.1 0.4 0.01
Joints:
- joint joint1: child cord1 -> string2; origin xyz=-0.02 0.0 0.12 rpy=1.57 0.0 0.0 -> xyz=-0.00585 0.0 0.0376 rpy=1.38 0.0 0.0
- joint joint2: child cord2 -> string1; origin xyz=-0.06 0.0 0.1 rpy=1.57 0.0 0.0 -> xyz=-0.01785 0.0 0.0278 rpy=1.38 0.0 0.0
- joint joint3: child cord3 -> string3; origin xyz=0.02 0.0 0.12 rpy=1.57 0.0 0.0 -> xyz=0.00585 0.0 0.0376 rpy=1.38 0.0 0.0
- joint joint4: child cord4 -> string4; origin xyz=0.06 0.0 0.1 rpy=1.57 0.0 0.0 -> xyz=0.01785 0.0 0.0278 rpy=1.38 0.0 0.0

Commit message: Add Python FSM and updated simviz config

File: urdf_models/flexiv_violin/violin.urdf (robot description, URDF)
Before this commit: robot violin, 5 links, 4 joints
Links:
- added link fake_link, mass 0.1; collision cylinder length=0.001 radius=0.001
Joints:
- added joint fake_joint: type prismatic, parent base_link, child fake_link, origin xyz=0.01785 0.0 0.0278 rpy=1.38 0.0 0.0, axis 0 0 1, limit lower=-2.7925 upper=2.7925 effort=123 velocity=2.0944
